Commit message: Filtrado, vamos tentar usar OM

File: traversability_mapping/urdf/sensor_box.urdf (robot description, URDF)
Before this commit: robot sensor_box, 23 links, 22 joints
Links:
- removed link base_link
- added link base_link2
Joints:
- joint base_link_to_base_sensor_box: parent base_link -> base_link2
- joint base_link_to_smatphone_frame: parent base_link -> base_link2
